File: output/porcupine/pcbs/porcupine.kicad_pcb (KiCad board)
At the start: 2 copper layers, 129.4 x 113.9 mm, 54 parts, among them J1 Jumper, J2 Jumper

Commit message: Beschreibung deiner Änderungen
Connections:
- D1 pad 2: P6 -> pinky_bottom
- D10 pad 2: P6 -> index_bottom
- D11 pad 2: P5 -> index_home
- D12 pad 2: P4 -> index_top
- D13 pad 2: P6 -> inner_bottom
- D14 pad 2: P5 -> inner_home
- D15 pad 2: P4 -> inner_top
- D16 pad 2: P7 -> near_thumb
- D17 pad 2: P7 -> home_thumb
- D18 pad 2: P7 -> far_thumb
- D2 pad 2: P5 -> pinky_home
- D3 pad 2: P4 -> pinky_top
- D4 pad 2: P6 -> ring_bottom
- D5 pad 2: P5 -> ring_home
- D6 pad 2: P4 -> ring_top
- D7 pad 2: P6 -> middle_bottom
- D8 pad 2: P5 -> middle_home
- D9 pad 2: P4 -> middle_top
Other:
- net class Default removed
- net class Power removed
