File: output/porcupine/pcbs/porcupine_top_plate.kicad_pcb (KiCad board)
At the start: 2 copper layers, 129.3 x 113.9 mm, 0 parts

Commit message: Beschreibung deiner Änderungen
Other:
- outline, holes or cut-outs redrawn
- net class Default removed
- net class Power removed
