File: output/porcupine_4thumb_keys/pcbs/porcupine_4thumb_keys.kicad_pcb (KiCad board)
At the start: 2 copper layers, 148.2 x 111.9 mm, 56 parts, among them J1 Jumper, J2 Jumper

Commit message: Beschreibung deiner Änderungen
Parts:
- moved D19 7.00 mm to (280.0, 175.7), turned to -45 degrees
- moved D18 6.87 mm to (263.8, 163.2), turned to -30 degrees
- moved S18 0.20 mm to (266.3, 158.9), turned to -30 degrees
- moved S19 0.07 mm to (283.5, 172.2), turned to -45 degrees
Connections:
- D1 pad 2: P6 -> pinky_bottom
- D10 pad 2: P6 -> index_bottom
- D11 pad 2: P5 -> index_home
- D12 pad 2: P4 -> index_top
- D13 pad 2: P6 -> inner_bottom
- D14 pad 2: P5 -> inner_home
- D15 pad 2: P4 -> inner_top
- D16 pad 2: P7 -> inner_thumb
- D17 pad 2: P7 -> near_thumb
- D18 pad 2: P7 -> home_thumb
- D19 pad 2: P7 -> far_thumb
- D2 pad 2: P5 -> pinky_home
- D3 pad 2: P4 -> pinky_top
- D4 pad 2: P6 -> ring_bottom
- D5 pad 2: P5 -> ring_home
- D6 pad 2: P4 -> ring_top
- D7 pad 2: P6 -> middle_bottom
- D8 pad 2: P5 -> middle_home
- D9 pad 2: P4 -> middle_top
Other:
- net class Default removed
- net class Power removed
