File: input/porcupine.kicad_pcb (KiCad board)
At the start: 2 copper layers, 144.8 x 104.6 mm, 31 parts, among them J1 Jumper, J2 Jumper

Commit message: Beschreibung deiner ÄnderungenOAO2
Parts:
- added D1: D_SOD-123, Diode_SMD:SOD-123, F.Cu at (176.5, 155.5)
- added D10: D_SOD-123, Diode_SMD:SOD-123, F.Cu at (227.4, 128.9)
- added D11: D_SOD-123, Diode_SMD:SOD-123, F.Cu at (227.4, 111.9)
- added D12: D_SOD-123, Diode_SMD:SOD-123, F.Cu at (227.4, 94.9)
- added D13: D_SOD-123, Diode_SMD:SOD-123, F.Cu at (246.4, 131.7)
- added D14: D_SOD-123, Diode_SMD:SOD-123, F.Cu at (246.4, 114.7)
- added D15: D_SOD-123, Diode_SMD:SOD-123, F.Cu at (246.4, 97.7)
- added D16: D_SOD-123, Diode_SMD:SOD-123, F.Cu at (241.2, 154.9)
- added D17: D_SOD-123, Diode_SMD:SOD-123, F.Cu at (260.8, 159.6)
- added D18: D_SOD-123, Diode_SMD:SOD-123, F.Cu at (278.5, 169.6)
- added D2: D_SOD-123, Diode_SMD:SOD-123, F.Cu at (171.5, 139.3)
- added D3: D_SOD-123, Diode_SMD:SOD-123, F.Cu at (166.6, 123.0)
- added D4: D_SOD-123, Diode_SMD:SOD-123, F.Cu at (190.2, 133.7)
- added D5: D_SOD-123, Diode_SMD:SOD-123, F.Cu at (187.2, 116.9)
- added D6: D_SOD-123, Diode_SMD:SOD-123, F.Cu at (184.3, 100.2)
- added D7: D_SOD-123, Diode_SMD:SOD-123, F.Cu at (208.1, 124.8)
- added D8: D_SOD-123, Diode_SMD:SOD-123, F.Cu at (206.9, 107.8)
- added D9: D_SOD-123, Diode_SMD:SOD-123, F.Cu at (205.6, 90.9)
- added MCU1: , ProMicro, F.Cu at (267.4, 103.7)
- added _2: , lib:bat2p0, F.Cu at (259.9, 129.7)
- added _3: , Button_Switch_SMD:SW_SPDT_PCM12, F.Cu at (277.3, 130.7)
- added _4_B: SW_Push, Button_Switch_SMD:SW_SPST_B3U-1000P, B.Cu at (262.4, 135.7)
- added _4_F: SW_Push, Button_Switch_SMD:SW_SPST_B3U-1000P, F.Cu at (262.4, 135.7)
- S1, S10, S11, S12, S13, S14, S15, S16, S17, S18, S2, S3, S4, S5, S6, S7, S8, S9: footprint Keyboards:Kailh_socket_PG1350_reversible_cropped_pads -> PG1350
- turned S1 to 17 degrees
- turned S10 to 0 degrees
- turned S12 to 0 degrees
- turned S13 to 0 degrees
- turned S14 to 0 degrees
- turned S15 to 0 degrees
- turned S16 to -6 degrees
- turned S17 to -21 degrees
- turned S18 to -38 degrees
- turned S2 to 17 degrees
- turned S3 to 17 degrees
- turned S4 to 10 degrees
- turned S5 to 10 degrees
- turned S6 to 10 degrees
- turned S8 to 5 degrees
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Routing:
- net ring_home: vias 1 -> 0
- net RST: vias 1 -> 0
- net RAW: vias 1 -> 0
- net GND: vias 2 -> 0
